Commit message: add scara4 and remove urdf_scara

File: scara4/urdf/scara4.urdf (robot description, URDF)
Before this commit: robot urdf_scara, 6 links, 5 joints
Links:
- removed link gripper
- link link1: mass 0.33397 -> 0.333965027627055; geometry collision mesh filename=package://scara4/meshes/link1.STL; visual mesh filename=package://scara4/meshes/link1.STL
- link link2: mass 0.34183 -> 0.341833276422222; geometry collision mesh filename=package://scara4/meshes/link2.STL; visual mesh filename=package://scara4/meshes/link2.STL
- link link3: mass 0.349496663604908 -> 0.349496704950288; geometry collision mesh filename=package://scara4/meshes/link3.STL; visual mesh filename=package://scara4/meshes/link3.STL
- link link4: mass 0.132586772624035 -> 0.132586780122943; geometry collision mesh filename=package://scara4/meshes/link4.STL; visual mesh filename=package://scara4/meshes/link4.STL
- link link5: mass 0.059264 -> 0.0592642341472502; geometry collision mesh filename=package://scara4/meshes/link5.STL; visual mesh filename=package://scara4/meshes/link5.STL
Joints:
- removed joint join5
- joint joint1: origin xyz=0 0 0.0408 rpy=1.5708 0 -0.78304 -> xyz=0 0 0.0408 rpy=1.5708 0 3.1416
- joint joint2: origin xyz=-4.5017E-05 0.17725 0.017 rpy=0 0 0 -> xyz=-4.5017E-05 0.097592 0.017 rpy=0 0 0
- joint joint3: origin xyz=4.5017E-05 0 -0.067 rpy=0 -1.2013 0 -> xyz=4.5017E-05 0 -0.067 rpy=0 0 0
- joint joint4: origin xyz=0 0 -0.1528 rpy=3.1416 0.39723 3.1416 -> xyz=0 0 -0.1528 rpy=3.1416 0 3.1416
